File: cad/impulse/impulse.kicad_pcb (KiCad board)
At the start: 8 copper layers, 138 parts, among them J1 Conn_02x04_Counter_Clockwise, J10 Conn_01x14_Socket, J11 DB125-2.54, J12 DB125-2.54, J13 Micro_SD_Card, J14 Conn_Coaxial, J2 DB125-2.54, J3 DB125-2.54, J4 Conn_01x06, J5 Conn_01x06, J6 Conn_01x06, J7 DB125-2.54, J8 GT-USB-7010ASV, J9 DB125-2.54, Q1 AO3415, SW1 SW_Push, U1 STM32G431CBUx, U10 BMI270, U11 W25Q32JVSS, U12 BGS12PL6, U13 SX1268, U2 MT2492, U3 MT2492, U4 LN2324DT2AG, U5 LN2324DT2AG, U6 USBLC6-2SC6, U7 LN2324DT2AG, U8 LN2324DT2AG, U9 HP203B, Y1 X252016MLB4SI, Y2 XL7EL89COI-111YLC-32M

Commit message: Modified oscillator circuit.
Parts:
- added R6: 47r, Resistor_SMD:R_0402_1005Metric, F.Cu at (148.2, 74.1)
- moved H1 13.3 mm to (89.3, 69.9)
- moved H2 13.3 mm to (89.3, 77.9)
- moved H3 13.3 mm to (89.3, 85.8)
- moved H4 13.3 mm to (89.3, 93.8)
- moved SW1 8.75 mm to (163.8, 87.7)
- moved U12 7.53 mm to (128.9, 121.4)
- renumbered R9 to R10, R10 to R11, R11 to R12, R12 to R13, R13 to R14, R14 to R15, R15 to R16, R16 to R17, R17 to R18, R18 to R19, R19 to R20, R20 to R21, R21 to R22, R22 to R23, R23 to R24, R24 to R25, R25 to R26, R26 to R27, R27 to R28, R28 to R29, R29 to R30, R30 to R31, R31 to R32, R32 to R33, R33 to R34, R34 to R35, R35 to R36, R36 to R37, R37 to R38, R6 to R7, R7 to R8, R8 to R9
Connections:
- C9 pad 1: /stm_xtb -> Net-(C9-Pad1)
- Y1 pad 1: /stm_xtb -> Net-(C9-Pad1)

Commit message: First layout.
Parts:
- removed J3: DB125-2.54, TerminalBlock_TE-Connectivity:TerminalBlock_TE_282834-2_1x02_P2.54mm_Horizontal
- removed JP1: Jumper_2_Open, Jumper:SolderJumper-2_P1.3mm_Bridged2Bar_Pad1.0x1.5mm
- removed R3, R4: 0r, Resistor_SMD:R_0402_1005Metric
- added R39: 100r, Resistor_SMD:R_0402_1005Metric, F.Cu at (164.5, 38.1)
- C13, C14, C15, C16, C17, C18, C19, C20, C24, C25, C4, C5, C6, C8, D1, D3, D4, D5, D6, D7, J13, L1, L2, R25, R7, U11, U2, U3, U6: moved to B.Cu
- J1: footprint Connector_PinHeader_1.27mm:PinHeader_2x04_P1.27mm_Vertical -> Connector_PinHeader_1.27mm:PinHeader_2x04_P1.27mm_Vertical_SMD
- R1: value 0r -> 1k5
- R10: value 13k3 -> 22k1; moved to B.Cu
- R11, R23: value 22k1 -> 13k3; moved to B.Cu
- R12: value 665r -> 22k1
- R13, R17, R19, R21: value 4k7 -> 665r
- R14: value 5k1 -> 4k7
- R16: value 665r -> 5k1
- R18, R20: value 665r -> 4k7
- R2: value 0r -> 1k5; moved to B.Cu
- R22: value 13k3 -> 4k7
- R24: value 1k5 -> 22k1
- R26: value 300r -> 1k5; moved to B.Cu
- R28: value 2k -> 300r
- R29: value 0r -> 2k; moved to B.Cu
- R31: value 300r -> 0r
- R32: value 13k3 -> 300r
- R36: value 140r -> 13k3
- R37: value 100r -> 140r
- R8: value 100k -> 0r
- R9: value 22k1 -> 100k; moved to B.Cu
- moved L9 78.2 mm to (138.2, 50.7)
- moved C44 78.2 mm to (151.8, 43.0)
- moved C45 78.2 mm to (151.8, 45.0)
- moved C37 77.9 mm to (122.3, 51.7)
- moved J2 77.3 mm to (164.2, 106.1), turned to -90 degrees
- moved H4 77.2 mm to (163.7, 114.5)
- moved C27 75.0 mm to (146.4, 44.6)
- moved H2 74.6 mm to (163.7, 72.0)
- moved L7 72.2 mm to (146.3, 41.6)
- moved D8 72.1 mm to (163.5, 76.7)
- moved C47 69.5 mm to (155.4, 59.9)
- moved C46 64.5 mm to (155.4, 63.6), turned to 180 degrees
- moved J4 64.4 mm to (156.3, 111.7), turned to -90 degrees
- moved C35 64.2 mm to (150.3, 73.1), turned to 180 degrees
- moved J5 62.9 mm to (156.3, 114.2), turned to -90 degrees
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Connections:
- C18 pad 1: Net-(JP1-A) -> +5V
- C19 pad 1: Net-(JP1-A) -> +5V
- C20 pad 1: Net-(JP1-A) -> +5V
- D1 pad 1: Net-(D1-K) -> vsense
- D2 pad 1: Net-(D1-K) -> vsense
- FB1 pad 1: Net-(D1-K) -> vsense
- J1 pad 2: Net-(J1-Pin_2) -> /stm_swdio
- J1 pad 3: Net-(J1-Pin_3) -> /stm_swclk
- J1 pad 6: Net-(J1-Pin_6) -> /usart2_tx
- J1 pad 7: Net-(J1-Pin_7) -> /usart2_rx
- L2 pad 2: Net-(JP1-A) -> +5V
- Q1 pad 2: Net-(D1-K) -> vsense
- R1 pad 1: /stm_swdio -> +3V3
- R1 pad 2: Net-(J1-Pin_2) -> fpc_scl
- R10 pad 1: Net-(U3-FB) -> Net-(U2-FB)
- R11 pad 1: Net-(D2-A) -> Net-(U3-FB)
- R12 pad 1: Net-(U4-G) -> Net-(D2-A)
- R12 pad 2: pyro_0 -> GND
- R13 pad 1: pyro_0 -> Net-(U4-G)
- R13 pad 2: GND -> pyro_0
- R14 pad 1: Net-(J8-CC1) -> pyro_0
- R15 pad 1: Net-(J8-CC2) -> Net-(J8-CC1)
- R16 pad 1: Net-(U5-G) -> Net-(J8-CC2)
- R16 pad 2: pyro_1 -> GND
- R17 pad 1: pyro_1 -> Net-(U5-G)
- R17 pad 2: GND -> pyro_1
- R18 pad 1: Net-(U7-G) -> pyro_1
- R18 pad 2: pyro_2 -> GND
- R19 pad 1: pyro_2 -> Net-(U7-G)
- R19 pad 2: GND -> pyro_2
- R2 pad 1: Net-(J1-Pin_7) -> +3V3
- R2 pad 2: /usart2_rx -> fpc_sda
- R20 pad 1: Net-(U8-G) -> pyro_2
- R20 pad 2: pyro_3 -> GND
- R21 pad 1: pyro_3 -> Net-(U8-G)
- R21 pad 2: GND -> pyro_3
- R22 pad 1: vbat_sense -> pyro_3
- R22 pad 2: VBUS -> GND
- R23 pad 1: +3V3 -> vbat_sense
- R23 pad 2: Net-(C21-Pad1) -> vsense
- R24 pad 2: i2c2_scl -> Net-(C21-Pad1)
- R25 pad 2: i2c2_sda -> i2c2_scl
- R26 pad 1: Net-(R26-Pad1) -> +3V3
- R26 pad 2: Net-(C21-Pad1) -> i2c2_sda
- R27 pad 1: Net-(C21-Pad1) -> Net-(R27-Pad1)
- R27 pad 2: button -> Net-(C21-Pad1)
- R28 pad 1: GND -> Net-(C21-Pad1)
- R28 pad 2: vbat_sense -> button
- R29 pad 2: Net-(U9-CSB) -> vbat_sense
- R30 pad 1: +3V3 -> GND
- R30 pad 2: Net-(U10-SDO) -> Net-(U9-CSB)
- R31 pad 1: Net-(D8-RK) -> +3V3
- R31 pad 2: led_r -> Net-(U10-SDO)
- R32 pad 1: +3V3 -> Net-(D8-RK)
- R32 pad 2: SD_cs -> led_r
- R33 pad 2: flash_mosi -> SD_cs
- R34 pad 2: flash_sck -> flash_mosi
- R35 pad 2: flash_miso -> flash_sck
- R36 pad 1: Net-(D8-GK) -> +3V3
- R36 pad 2: led_g -> flash_miso
- R37 pad 1: Net-(D8-BK) -> Net-(D8-GK)
- R37 pad 2: led_b -> led_g
- R38 pad 1: /Connectivity/sx_dio_2 -> Net-(D8-BK)
- R38 pad 2: Net-(U12-CTRL) -> led_b
- R8 pad 1: Net-(JP1-A) -> vinp
- R8 pad 2: Net-(U3-FB) -> Net-(U3-EN)
- R9 pad 1: Net-(U2-FB) -> +5V
- R9 pad 2: GND -> Net-(U3-FB)
- SW1 pad 2: Net-(R26-Pad1) -> Net-(R27-Pad1)
- U3 pad 4: vinp -> Net-(U3-EN)
Routing:
- net GND: track 0.00 -> 115.0 mm, vias 0 -> 75
- net +3V3: track 0.00 -> 65.5 mm, vias 0 -> 15
- net +5V: track 0.00 -> 57.4 mm, vias 0 -> 2
- net VBUS: track 0.00 -> 55.8 mm, vias 0 -> 19
- net vinp: track 0.00 -> 45.7 mm, vias 0 -> 9
- net button: track 0.00 -> 38.2 mm, vias 0 -> 3
- net flash_miso: track 0.00 -> 34.9 mm, vias 0 -> 3
- net servo_5: track 0.00 -> 33.1 mm, vias 0 -> 2
- net usb_d-: track 0.00 -> 32.9 mm, vias 0 -> 2
- net pyro_1: track 0.00 -> 32.7 mm, vias 0 -> 3
- net usb_d+: track 0.00 -> 31.7 mm, vias 0 -> 2
- net servo_0: track 0.00 -> 31.1 mm, vias 0 -> 2
- net /usart2_tx: track 0.00 -> 30.8 mm, vias 0 -> 2
- net servo_1: track 0.00 -> 30.2 mm, vias 0 -> 2
- net servo_3: track 0.00 -> 29.9 mm, vias 0 -> 2
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- added copper zone on In3.Cu, net +3V3
- added copper zone on In1.Cu, net GND
- added copper zone on In4.Cu, net GND
- added copper zone on In6.Cu, net GND
- added copper zone on B.Cu, net VBUS
- added copper zone on F.Cu, net VBUS
Other:
- board outline added: 35 x 50 mm

Commit message: Final version, ordered it.
Parts:
- added G***: LOGO, LOGO, F.Cu at (144.8, 81.8)
- added G***: LOGO, LOGO, B.Cu at (151.8, 95.2)
- added kibuzzard-647A5142: G***, kibuzzard-647A5142, F.Cu at (155.6, 79.7)
- C11, C12, C26, C3, C37, C44, C45, L7, L9, R1, R13, R14, R17, R18, R19, R20, R21, R22, R8: moved to B.Cu
- C27, C28, C29, C30, C31, C32, C33, C34, C36, C38, C39, C40, C41, C42, C43: footprint Capacitor_SMD:C_0402_1005Metric -> Capacitor_SMD:C_0201_0603Metric
- C35: footprint Capacitor_SMD:C_0603_1608Metric -> Capacitor_SMD:C_0201_0603Metric
- L3, L4, L5, L6, L8: footprint Inductor_SMD:L_0402_1005Metric -> Inductor_SMD:L_0201_0603Metric
- U4, U5, U7, U8: value LN2324DT2AG -> G2014; moved to B.Cu
- moved R39 39.5 mm to (146.6, 73.4)
- moved C37 38.8 mm to (154.7, 72.9), turned to 90 degrees
- moved L7 34.7 mm to (159.1, 73.8), turned to 90 degrees
- moved C44 31.0 mm to (156.5, 73.7), turned to 90 degrees
- moved L9 29.9 mm to (157.8, 73.2), turned to 90 degrees
- moved C27 28.6 mm to (147.4, 73.2), turned to -90 degrees
- moved C45 26.7 mm to (157.6, 71.0), turned to 180 degrees
- moved R2 20.1 mm to (137.4, 101.2), turned to 0 degrees
- moved C47 16.3 mm to (154.1, 76.1), turned to 90 degrees
- moved Y2 14.4 mm to (156.0, 76.1), turned to 180 degrees
- moved C46 12.8 mm to (157.9, 76.1), turned to -90 degrees
- moved C16 8.48 mm to (136.3, 105.5), turned to 90 degrees
- moved L3 7.00 mm to (152.5, 73.3), turned to 0 degrees
- moved C31 6.45 mm to (152.5, 72.5), turned to 180 degrees
- moved C29 5.88 mm to (152.2, 74.3), turned to -90 degrees
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Connections:
- J4 pad 1: servo_0 -> servo_3
- J4 pad 3: servo_2 -> servo_0
- J4 pad 4: servo_3 -> servo_2
Routing:
- net GND: track 115.0 -> 275.6 mm, vias 75 -> 162
- net vbat_sense: track 6.26 -> 59.2 mm, vias 0 -> 2
- net fpc_gpio: track 5.38 -> 39.7 mm, vias 1 -> 2
- net sx_nss: track 1.84 -> 33.5 mm, vias 1 -> 4
- net sx_sck: track 2.28 -> 31.2 mm, vias 1 -> 2
- net sx_miso: track 1.67 -> 29.2 mm, vias 1 -> 2
- net servo_5: track 33.1 -> 58.1 mm
- net VBUS: track 55.8 -> 80.8 mm, vias 19 -> 9
- net sx_mosi: track 3.24 -> 28.1 mm, vias 1 -> 2
- net fpc_sda: track 6.99 -> 26.1 mm, vias 1 -> 2
- net fpc_mosi: track 20.6 -> 38.3 mm, vias 0 -> 2
- net /Connectivity/sx_dio_2: track 0.00 -> 17.6 mm, vias 0 -> 2
- net fpc_tx: track 1.34 -> 17.4 mm, vias 1 -> 0
- net +5V: track 57.4 -> 42.5 mm, vias 2 -> 0
- net fpc_miso: track 18.1 -> 30.0 mm, vias 0 -> 2
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- added copper zone on B.Cu, net GND
- added copper zone on F.Cu, net GND
- removed copper zone on B.Cu, net VBUS
- removed copper zone on F.Cu, net VBUS
Other:
- board text added: "JLCJLCJLCJLC"
