File: cad/impulse/power-domain.kicad_sch (KiCad schematic)
At the start: 24 parts, among them Q101 AO3415, U2 MT2492, U3 MT2492

Commit message: First layout.
Parts:
- removed JP101: Jumper_2_Open, Jumper:SolderJumper-2_P1.3mm_Bridged2Bar_Pad1.0x1.5mm, symbol Jumper:Jumper_2_Open
- added R8: 0r, Resistor_SMD:R_0402_1005Metric, symbol Device:R_Small
- renumbered R9 to R10, R10 to R11, R8 to R9
Connections:
- net +5V: now also C18.1, C19.1, C20.1, L2.2, R9.1
- net vinp: now also R8.1; no longer U3.4 (EN)
- net vsense: now reaches D1.1 (K), D2.1 (K), FB1.1, Q101.2 (S)
- new net: R8.2, U3.4 (EN)
Changed lines of the file:
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@@
   (junction (at 236.22 29.21) (diameter 0) (color 0 0 0 0)
   )
+  (junction (at 53.34 30.48) (diameter 0) (color 0 0 0 0)
+  )
   (junction (at 119.38 29.21) (diameter 0) (color 0 0 0 0)
   )
   (junction (at 127 29.21) (diameter 0) (color 0 0 0 0)
   )
-  (junction (at 201.93 29.21) (diameter 0) (color 0 0 0 0)
-  )
   (junction (at 148.59 29.21) (diameter 0) (color 0 0 0 0)
   )
@@
   (junction (at 102.87 29.21) (diameter 0) (color 0 0 0 0)
   )
+  (junction (at 200.66 29.21) (diameter 0) (color 0 0 0 0)
+  )
   (junction (at 127 34.29) (diameter 0) (color 0 0 0 0)
   )
@@
     (stroke (width 0) (type default))
   )
-  (wire (pts (xy 195.58 29.21) (xy 201.93 29.21))
+  (wire (pts (xy 195.58 29.21) (xy 200.66 29.21))
     (stroke (width 0) (type default))
   )
@@
     (stroke (width 0) (type default))
   )
-  (wire (pts (xy 48.26 30.48) (xy 55.88 30.48))
-    (stroke (width 0) (type default))
-  )
-  (wire (pts (xy 201.93 34.29) (xy 201.93 29.21))
+  (wire (pts (xy 48.26 30.48) (xy 53.34 30.48))
+    (stroke (width 0) (type default))
+  )
+  (wire (pts (xy 200.66 34.29) (xy 203.2 34.29))
+    (stroke (width 0) (type default))
+  )
+  (wire (pts (xy 53.34 30.48) (xy 55.88 30.48))
     (stroke (width 0) (type default))
   )
@@
     (stroke (width 0) (type default))
   )
-  (wire (pts (xy 203.2 34.29) (xy 201.93 34.29))
-    (stroke (width 0) (type default))
-  )
   (wire (pts (xy 102.87 34.29) (xy 102.87 29.21))
     (stroke (width 0) (type default))
@@
     (stroke (width 0) (type default))
   )
-  (wire (pts (xy 251.46 29.21) (xy 254 29.21))
+  (wire (pts (xy 251.46 29.21) (xy 257.81 29.21))
     (stroke (width 0) (type default))
   )
@@
     (stroke (width 0) (type default))
   )
+  (wire (pts (xy 53.34 30.48) (xy 53.34 34.29))
+    (stroke (width 0) (type default))
+  )
   (wire (pts (xy 38.1 38.1) (xy 45.72 38.1))
     (stroke (width 0) (type default))
@@
     (stroke (width 0) (type default))
   )
-  (wire (pts (xy 201.93 29.21) (xy 203.2 29.21))
+  (wire (pts (xy 200.66 29.21) (xy 203.2 29.21))
     (stroke (width 0) (type default))
   )
@@
     )
   )
+  (global_label "vsense" (shape input) (at 53.34 34.29 0) (fields_autoplaced)
+    (effects (font (size 1.27 1.27)) (justify left))
+    (property "Intersheetrefs" "${INTERSHEET_REFS}" (at 62.5958 34.29 0)
+      (effects (font (size 1.27 1.27)) (justify left) hide)
+    )
+  )
   (global_label "vinp" (shape input) (at 64.77 30.48 0) (fields_autoplaced)
     (effects (font (size 1.27 1.27)) (justify left))
@@
   (symbol (lib_id "Device:R_Small") (at 127 36.83 0) (unit 1)
     (in_bom yes) (on_board yes) (dnp no)
-    (property "Reference" "R9" (at 128.27 35.56 0)
+    (property "Reference" "R10" (at 128.27 35.56 0)
       (effects (font (size 1.27 1.27)) (justify left))
     )
@@
       (project "impulse"
         (path "/eb4cfece-5fcb-437a-ac58-337ab6512039/8b8b63e5-7f69-4185-825a-2602e0d2cd2e"
-          (reference "R9") (unit 1)
+          (reference "R10") (unit 1)
         )
       )
@@
     )
   )
-  (symbol (lib_id "power:+5V") (at 264.16 29.21 0) (unit 1)
-    (in_bom yes) (on_board yes) (dnp no) (fields_autoplaced)
-    (property "Reference" "#PWR015" (at 264.16 33.02 0)
-      (effects (font (size 1.27 1.27)) hide)
-    )
-    (property "Value" "+5V" (at 264.16 25.4 0)
-      (effects (font (size 1.27 1.27)))
-    )
-    (property "Footprint" "" (at 264.16 29.21 0)
-      (effects (font (size 1.27 1.27)) hide)
-    )
-    (property "Datasheet" "" (at 264.16 29.21 0)
+  (symbol (lib_id "power:+5V") (at 257.81 29.21 0) (unit 1)
+    (in_bom yes) (on_board yes) (dnp no) (fields_autoplaced)
+    (property "Reference" "#PWR015" (at 257.81 33.02 0)
+      (effects (font (size 1.27 1.27)) hide)
+    )
+    (property "Value" "+5V" (at 257.81 25.4 0)
+      (effects (font (size 1.27 1.27)))
+    )
+    (property "Footprint" "" (at 257.81 29.21 0)
+      (effects (font (size 1.27 1.27)) hide)
+    )
+    (property "Datasheet" "" (at 257.81 29.21 0)
       (effects (font (size 1.27 1.27)) hide)
     )
@@
       (project "impulse"
         (path "/eb4cfece-5fcb-437a-ac58-337ab6512039/8b8b63e5-7f69-4185-825a-2602e0d2cd2e"
-          (reference "R11") (unit 1)
+          (reference "R12") (unit 1)
         )
       )
@@
     )
   )
-  (symbol (lib_id "Jumper:Jumper_2_Open") (at 259.08 29.21 0) (unit 1)
-    (in_bom yes) (on_board yes) (dnp no)
-    (property "Reference" "JP101" (at 261.62 31.75 0)
-      (effects (font (size 1.27 1.27)))
-    )
-    (property "Value" "Jumper_2_Open" (at 261.62 34.29 0)
-      (effects (font (size 1.27 1.27)))
-    )
-    (property "Footprint" "Jumper:SolderJumper-2_P1.3mm_Bridged2Bar_Pad1.0x1.5mm" (at 259.08 29.21 0)
-      (effects (font (size 1.27 1.27)) hide)
-    )
-    (property "Datasheet" "~" (at 259.08 29.21 0)
-      (effects (font (size 1.27 1.27)) hide)
-    )
-    (property "lcsc" "" (at 259.08 29.21 0)
-      (effects (font (size 1.27 1.27)) hide)
-    )
-    (pin "1")
-    (pin "2")
-    (instances
-      (project "valentine"
-        (path "/1e598ca5-0882-4bb6-9d64-e7e7f53f92db"
-          (reference "JP101") (unit 1)
-        )
-      )
-      (project "impulse"
-        (path "/eb4cfece-5fcb-437a-ac58-337ab6512039/8b8b63e5-7f69-4185-825a-2602e0d2cd2e"
-          (reference "JP1") (unit 1)
-        )
-      )
-    )
-  )
   (symbol (lib_id "Device:C_Small") (at 215.9 24.13 90) (unit 1)
     (in_bom yes) (on_board yes) (dnp no)
@@
   (symbol (lib_id "Device:R_Small") (at 226.06 36.83 0) (unit 1)
     (in_bom yes) (on_board yes) (dnp no)
-    (property "Reference" "R10" (at 227.33 35.56 0)
+    (property "Reference" "R11" (at 227.33 35.56 0)
       (effects (font (size 1.27 1.27)) (justify left))
     )
@@
       (project "impulse"
         (path "/eb4cfece-5fcb-437a-ac58-337ab6512039/8b8b63e5-7f69-4185-825a-2602e0d2cd2e"
-          (reference "R10") (unit 1)
+          (reference "R11") (unit 1)
         )
       )
@@
   (symbol (lib_id "Device:R_Small") (at 226.06 31.75 0) (unit 1)
     (in_bom yes) (on_board yes) (dnp no)
-    (property "Reference" "R8" (at 227.33 31.115 0)
+    (property "Reference" "R9" (at 227.33 31.115 0)
       (effects (font (size 1.27 1.27)) (justify left))
     )
@@
       (project "impulse"
         (path "/eb4cfece-5fcb-437a-ac58-337ab6512039/8b8b63e5-7f69-4185-825a-2602e0d2cd2e"
-          (reference "R8") (unit 1)
+          (reference "R9") (unit 1)
         )
       )
@@
         )
       )
+    )
+  )
+  (symbol (lib_id "Device:R_Small") (at 200.66 31.75 0) (unit 1)
+    (in_bom yes) (on_board yes) (dnp no)
+    (property "Reference" "R8" (at 199.39 36.83 0)
+      (effects (font (size 1.27 1.27)) (justify left))
+    )
+    (property "Value" "0r" (at 199.39 39.37 0)
+      (effects (font (size 1.27 1.27)) (justify left))
+    )
+    (property "Footprint" "Resistor_SMD:R_0402_1005Metric" (at 200.66 31.75 0)
+      (effects (font (size 1.27 1.27)) hide)
+    )
+    (property "Datasheet" "~" (at 200.66 31.75 0)
+      (effects (font (size 1.27 1.27)) hide)
+    )
+    (pin "1")
+    (pin "2")
+    (instances
+      (project "impulse"
+        (path "/eb4cfece-5fcb-437a-ac58-337ab6512039/8b8b63e5-7f69-4185-825a-2602e0d2cd2e"
+          (reference "R8") (unit 1)
+        )
+      )

Commit message: Final version, ordered it.
Parts:
- R8: lcsc (none) -> C21376
Changed lines of the file:
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@@
+      (effects (font (size 1.27 1.27)) hide)
+    )
+    (property "lcsc" "C21376" (at 200.66 31.75 0)
       (effects (font (size 1.27 1.27)) hide)
     )
